File: bling mx/pulso - bling mx.kicad_pcb (KiCad board)
At the start: 2 copper layers, 229.6 x 95.2 mm, 101 parts, among them J1 MJ-4PP-9, J2 MJ-4PP-9, SW2 SW_Push, SW20 SW_Push, SW21 SW_Push, U2 xiao-ble

Commit message: Add files via upload
Parts:
- added ?: , , F.Cu at (170.4, 74.5)
- added ?: , , F.Cu at (150.0, 74.6)
- added ?: , , B.Cu at (161.4, 74.5)
- added ?: , , B.Cu at (140.9, 74.5)
- added BT1: Device_Battery_Cell, pierce:BatteryHolder_Keystone_3034_1x20mm, F.Cu at (144.4, 87.1)
- added BT1: Device_Battery_Cell, pierce:BatteryHolder_Keystone_3034_1x20mm, F.Cu at (164.9, 87.1)
- added PWR: SW_SPDT, TOTEMlib:MSK12C02, F.Cu at (162.4, 103.7)
- added PWR: SW_SPDT, TOTEMlib:MSK12C02, F.Cu at (141.9, 103.7)
- added U1: ProMicro, swoop:ProMicro_jumpers, F.Cu at (145.4, 88.7)
- added U1: ProMicro, swoop:ProMicro_jumpers, F.Cu at (281.5, 91.5)
- added U1: ProMicro, swoop:ProMicro_jumpers, F.Cu at (30.0, 91.9)
- added U1: ProMicro, swoop:ProMicro_jumpers, F.Cu at (165.8, 88.7)
- added mouse-bite-2mm-slot2: VAL**, Duckyb-Parts:mouse-bite-5mm-slot-with-space-for-track, F.Cu at (176.1, 93.7)
- added mouse-bite-2mm-slot2: VAL**, Duckyb-Parts:mouse-bite-5mm-slot-with-space-for-track, F.Cu at (135.2, 77.0)
- added mouse-bite-2mm-slot2: VAL**, Duckyb-Parts:mouse-bite-5mm-slot-with-space-for-track, F.Cu at (176.1, 77.0)
- added mouse-bite-2mm-slot2: VAL**, Duckyb-Parts:mouse-bite-5mm-slot-with-space-for-track, F.Cu at (135.1, 93.3)
- ?: moved to B.Cu
- moved BatGND1 32.6 mm to (278.3, 99.6)
- moved DL10 27.4 mm to (263.5, 88.2)
- moved J1 27.4 mm to (288.4, 112.6)
- moved Mounting 02 27.4 mm to (281.2, 119.1)
- moved PWR 27.4 mm to (271.9, 63.3)
- moved SW2 27.4 mm to (263.0, 59.9)
- moved ? 27.4 mm to (273.3, 109.6)
- moved BT1 27.4 mm to (224.6, 110.9)
- moved Bat+r1 27.4 mm to (278.4, 102.9)
- moved D16 27.4 mm to (243.6, 119.9)
- moved DL1 27.4 mm to (187.2, 80.1)
- moved DL11 27.4 mm to (187.0, 117.4)
- moved DL12 27.4 mm to (206.0, 106.1)
- moved DL13 27.4 mm to (225.1, 100.8)
- moved DL14 27.4 mm to (243.8, 104.0)
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Routing:
- net (no net): track 0.00 -> 156.3 mm, vias 0 -> 4
- net GND_R: track 36.6 -> 70.0 mm, vias 1 -> 2
- net RESET_R: track 47.4 -> 73.5 mm
- net BAT+_L: track 25.9 -> 45.1 mm, vias 1 -> 2
- net Net-(DL5-Pad2): track 0.00 -> 17.3 mm, vias 0 -> 1
- net BAT+_R: track 54.1 -> 67.7 mm
- net RESET_L: track 70.0 -> 82.8 mm
- net GND_L: track 58.8 -> 71.0 mm
- net VBAT_L: track 106.8 -> 114.4 mm
- net VBAT_R: track 193.8 -> 201.1 mm
- net TX_R: track 35.5 -> 31.7 mm
- net COL3_L: track 142.4 -> 144.7 mm
- net ROW3_R: track 89.6 -> 91.7 mm
- net COL0_R: track 177.3 -> 175.2 mm
- net COL0_L: track 182.5 -> 180.8 mm
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Other:
- board size 229.6 x 95.2 mm -> 270.6 x 95.6 mm
- board text added: "left"
- board text added: "right"

Commit message: Add files via upload
Parts:
- G***: moved to F.Cu
- moved G*** 7.76 mm to (154.9, 93.2), turned to 0 degrees

Commit message: Add files via upload
Parts:
- removed the G*** at (154.9, 93.2)
- moved BT1 2.00 mm to (166.9, 87.1)
