File: swoo/pulso novo.kicad_pcb (KiCad board)
At the start: 2 copper layers, 242.8 x 99.3 mm, 100 parts, among them SW1 MX, SW17 MX, SW18 MX, U2 xiao-ble

Commit message: Add files via upload
Parts:
- removed the ? at (204.7, 101.3)
- removed the ? at (182.3, 67.4)
- removed the ? at (169.4, 112.2)
- removed the ? at (236.5, 107.1)
- removed the ? at (242.6, 55.7)
- removed Bat+r1 (x2), BatGND1 (x2): MountingHole_Pad, kbd:1pin_conn
- removed RSW1 (x2): SW_PUSH, kbd:ResetSW
- removed the Ref** at (160.7, 106.8)
- removed the Ref** at (146.4, 114.0)
- removed SW1 (x32), SW17 (x2), SW18 (x2): MX, swoop:MX_socket_reversible
- removed the U2 at (152.5, 59.0)
- removed mouse-bite-2mm-slot2 (x2): VAL**, Duckyb-Parts:mouse-bite-5mm-slot-with-space-for-track
- added ?: , clipboard:f92b4755-0677-424b-a33d-44c3fe197dca, F.Cu at (136.8, 80.4)
- added ?: , clipboard:f92b4755-0677-424b-a33d-44c3fe197dca, F.Cu at (140.6, 80.3)
- added ?: , , B.Cu at (140.7, 80.6)
- added JP1: Jumper_2_Open, Jumper:SolderJumper-2_P1.3mm_Open_RoundedPad1.0x1.5mm, F.Cu at (122.1, 50.3)
- added JP1: Jumper_2_Open, Jumper:SolderJumper-2_P1.3mm_Open_RoundedPad1.0x1.5mm, F.Cu at (146.2, 50.2)
- added JP2: Jumper_2_Open, Jumper:SolderJumper-2_P1.3mm_Open_RoundedPad1.0x1.5mm, F.Cu at (122.1, 52.8)
- added JP2: Jumper_2_Open, Jumper:SolderJumper-2_P1.3mm_Open_RoundedPad1.0x1.5mm, F.Cu at (146.2, 52.7)
- added JP3: Jumper_2_Open, Jumper:SolderJumper-2_P1.3mm_Open_RoundedPad1.0x1.5mm, F.Cu at (146.2, 55.2)
- added JP3: Jumper_2_Open, Jumper:SolderJumper-2_P1.3mm_Open_RoundedPad1.0x1.5mm, F.Cu at (122.1, 55.3)
- added JP4: Jumper_2_Open, Jumper:SolderJumper-2_P1.3mm_Open_RoundedPad1.0x1.5mm, F.Cu at (122.1, 57.8)
- added JP4: Jumper_2_Open, Jumper:SolderJumper-2_P1.3mm_Open_RoundedPad1.0x1.5mm, F.Cu at (146.2, 57.7)
- added JP5: Jumper_2_Open, Jumper:SolderJumper-2_P1.3mm_Open_RoundedPad1.0x1.5mm, F.Cu at (136.9, 64.5)
- added JP5: Jumper_2_Open, Jumper:SolderJumper-2_P1.3mm_Open_RoundedPad1.0x1.5mm, F.Cu at (132.3, 64.5)
- added JP5: Jumper_2_Open, Jumper:SolderJumper-2_P1.3mm_Open_RoundedPad1.0x1.5mm, B.Cu at (146.2, 50.2)
- added JP5: Jumper_2_Open, Jumper:SolderJumper-2_P1.3mm_Open_RoundedPad1.0x1.5mm, B.Cu at (122.1, 50.3)
- added JP5: Jumper_2_Open, Jumper:SolderJumper-2_P1.3mm_Open_RoundedPad1.0x1.5mm, B.Cu at (136.9, 64.5)
- added JP5: Jumper_2_Open, Jumper:SolderJumper-2_P1.3mm_Open_RoundedPad1.0x1.5mm, B.Cu at (132.3, 64.5)
- added JP6: Jumper_2_Open, Jumper:SolderJumper-2_P1.3mm_Open_RoundedPad1.0x1.5mm, B.Cu at (146.2, 52.7)
- added JP6: Jumper_2_Open, Jumper:SolderJumper-2_P1.3mm_Open_RoundedPad1.0x1.5mm, B.Cu at (122.1, 52.8)
- added JP7: Jumper_2_Open, Jumper:SolderJumper-2_P1.3mm_Open_RoundedPad1.0x1.5mm, B.Cu at (146.2, 55.2)
- added JP7: Jumper_2_Open, Jumper:SolderJumper-2_P1.3mm_Open_RoundedPad1.0x1.5mm, B.Cu at (122.1, 55.3)
- added JP8: Jumper_2_Open, Jumper:SolderJumper-2_P1.3mm_Open_RoundedPad1.0x1.5mm, F.Cu at (146.2, 62.7)
- added JP8: Jumper_2_Open, Jumper:SolderJumper-2_P1.3mm_Open_RoundedPad1.0x1.5mm, B.Cu at (146.2, 62.7)
- added JP8: Jumper_2_Open, Jumper:SolderJumper-2_P1.3mm_Open_RoundedPad1.0x1.5mm, B.Cu at (122.1, 62.8)
- added JP8: Jumper_2_Open, Jumper:SolderJumper-2_P1.3mm_Open_RoundedPad1.0x1.5mm, B.Cu at (122.0, 65.3)
- added JP8: Jumper_2_Open, Jumper:SolderJumper-2_P1.3mm_Open_RoundedPad1.0x1.5mm, B.Cu at (122.1, 57.8)
- added JP8: Jumper_2_Open, Jumper:SolderJumper-2_P1.3mm_Open_RoundedPad1.0x1.5mm, B.Cu at (146.1, 65.2)
- added JP8: Jumper_2_Open, Jumper:SolderJumper-2_P1.3mm_Open_RoundedPad1.0x1.5mm, F.Cu at (146.2, 60.2)
- added JP8: Jumper_2_Open, Jumper:SolderJumper-2_P1.3mm_Open_RoundedPad1.0x1.5mm, F.Cu at (122.1, 65.3)
- added JP8: Jumper_2_Open, Jumper:SolderJumper-2_P1.3mm_Open_RoundedPad1.0x1.5mm, F.Cu at (122.1, 60.3)
- added JP8: Jumper_2_Open, Jumper:SolderJumper-2_P1.3mm_Open_RoundedPad1.0x1.5mm, F.Cu at (122.1, 62.8)
- added JP8: Jumper_2_Open, Jumper:SolderJumper-2_P1.3mm_Open_RoundedPad1.0x1.5mm, F.Cu at (146.2, 65.2)
- added JP8: Jumper_2_Open, Jumper:SolderJumper-2_P1.3mm_Open_RoundedPad1.0x1.5mm, B.Cu at (146.2, 60.2)
- added JP8: Jumper_2_Open, Jumper:SolderJumper-2_P1.3mm_Open_RoundedPad1.0x1.5mm, B.Cu at (146.2, 57.7)
- added JP8: Jumper_2_Open, Jumper:SolderJumper-2_P1.3mm_Open_RoundedPad1.0x1.5mm, B.Cu at (122.1, 60.3)
- added RST_B: SW_Push, kbd:SW_SPST_B3U-1000P, F.Cu at (148.7, 83.8)
- added RST_B: SW_Push, kbd:SW_SPST_B3U-1000P, B.Cu at (148.7, 83.8)
- added SW14: SW_Push, Keyswitches by Daprice:Kailh_socket_MX_reversible_sameside, F.Cu at (31.2, 106.6)
- added SW14: SW_Push, Keyswitches by Daprice:Kailh_socket_MX_reversible_sameside, F.Cu at (88.4, 57.0)
- added SW14: SW_Push, Keyswitches by Daprice:Kailh_socket_MX_reversible_sameside, F.Cu at (82.6, 115.8)
- added SW14: SW_Push, Keyswitches by Daprice:Kailh_socket_MX_reversible_sameside, F.Cu at (107.4, 78.6)
- added SW14: SW_Push, Keyswitches by Daprice:Kailh_socket_MX_reversible_sameside, F.Cu at (31.2, 68.5)
- added SW14: SW_Push, Keyswitches by Daprice:Kailh_socket_MX_reversible_sameside, F.Cu at (107.4, 97.6)
- added SW14: SW_Push, Keyswitches by Daprice:Kailh_socket_MX_reversible_sameside, F.Cu at (69.3, 69.6)
- added SW14: SW_Push, Keyswitches by Daprice:Kailh_socket_MX_reversible_sameside, F.Cu at (69.3, 50.5)
- added SW14: SW_Push, Keyswitches by Daprice:Kailh_socket_MX_reversible_sameside, B.Cu at (69.3, 88.6)
- added SW14: SW_Push, Keyswitches by Daprice:Kailh_socket_MX_reversible_sameside, B.Cu at (31.2, 106.6)
- added SW14: SW_Push, Keyswitches by Daprice:Kailh_socket_MX_reversible_sameside, B.Cu at (82.6, 115.8)
- added SW14: SW_Push, Keyswitches by Daprice:Kailh_socket_MX_reversible_sameside, F.Cu at (50.3, 94.6)
- added SW14: SW_Push, Keyswitches by Daprice:Kailh_socket_MX_reversible_sameside, B.Cu at (107.4, 97.6)
- added SW14: SW_Push, Keyswitches by Daprice:Kailh_socket_MX_reversible_sameside, B.Cu at (50.3, 94.6)
- added SW14: SW_Push, Keyswitches by Daprice:Kailh_socket_MX_reversible_sameside, B.Cu at (50.3, 75.6)
- added SW14: SW_Push, Keyswitches by Daprice:Kailh_socket_MX_reversible_sameside, B.Cu at (69.3, 50.5)
- added SW14: SW_Push, Keyswitches by Daprice:Kailh_socket_MX_reversible_sameside, B.Cu at (107.4, 59.5)
- added SW14: SW_Push, Keyswitches by Daprice:Kailh_socket_MX_reversible_sameside, B.Cu at (88.4, 57.0)
- added SW14: SW_Push, Keyswitches by Daprice:Kailh_socket_MX_reversible_sameside, B.Cu at (88.4, 76.1)
- added SW14: SW_Push, Keyswitches by Daprice:Kailh_socket_MX_reversible_sameside, B.Cu at (88.4, 95.1)
- added SW14: SW_Push, Keyswitches by Daprice:Kailh_socket_MX_reversible_sameside, B.Cu at (107.4, 78.6)
- added SW14: SW_Push, Keyswitches by Daprice:Kailh_socket_MX_reversible_sameside, B.Cu at (50.3, 56.5)
- added SW14: SW_Push, Keyswitches by Daprice:Kailh_socket_MX_reversible_sameside, F.Cu at (107.4, 59.5)
- added SW14: SW_Push, Keyswitches by Daprice:Kailh_socket_MX_reversible_sameside, B.Cu at (69.3, 69.6)
- added SW14: SW_Push, Keyswitches by Daprice:Kailh_socket_MX_reversible_sameside, B.Cu at (31.2, 87.6)
- added SW14: SW_Push, Keyswitches by Daprice:Kailh_socket_MX_reversible_sameside, B.Cu at (31.2, 68.5)
- added SW14: SW_Push, Keyswitches by Daprice:Kailh_socket_MX_reversible_sameside, F.Cu at (50.3, 75.6)
- added SW14: SW_Push, Keyswitches by Daprice:Kailh_socket_MX_reversible_sameside, F.Cu at (31.2, 87.6)
- added SW14: SW_Push, Keyswitches by Daprice:Kailh_socket_MX_reversible_sameside, F.Cu at (88.4, 76.1)
- added SW14: SW_Push, Keyswitches by Daprice:Kailh_socket_MX_reversible_sameside, F.Cu at (50.3, 56.5)
- added SW14: SW_Push, Keyswitches by Daprice:Kailh_socket_MX_reversible_sameside, F.Cu at (69.3, 88.6)
- added SW14: SW_Push, Keyswitches by Daprice:Kailh_socket_MX_reversible_sameside, F.Cu at (88.4, 95.1)
- added SW20 (x2): SW_Push, Keyswitches by Daprice:Kailh_socket_MX_reversible_sameside, F.Cu at (124.1, 129.2)
- added SW21 (x2): SW_Push, Keyswitches by Daprice:Kailh_socket_MX_reversible_sameside, F.Cu at (104.3, 120.0)
- BT1, D16, D17, D18, DL1, DL10, DL11, DL12, DL13, DL14, DL15, DL2, DL3, DL4, DL5, DL6, DL7, DL8, DL9, PWR: moved to B.Cu
- moved DL1 218.1 mm to (31.1, 78.3), turned to 180 degrees
- moved DL6 218.0 mm to (31.2, 97.2), turned to 180 degrees
- moved DL11 218.0 mm to (31.2, 116.3), turned to 180 degrees
- moved DL12 179.8 mm to (50.3, 104.2), turned to 180 degrees
- moved DL7 179.8 mm to (50.3, 84.9), turned to 180 degrees
- moved DL2 179.8 mm to (50.4, 66.0), turned to 180 degrees
- moved DL3 141.8 mm to (69.2, 60.0), turned to 180 degrees
- moved DL8 141.7 mm to (69.3, 79.2), turned to 180 degrees
- moved DL13 141.6 mm to (69.5, 98.3), turned to 180 degrees
- moved D16 127.4 mm to (92.4, 111.2)
- moved D17 122.9 mm to (94.6, 111.2)
- moved D18 118.5 mm to (96.8, 111.2)
- moved DL4 103.7 mm to (88.4, 66.4), turned to 180 degrees
- moved DL9 103.6 mm to (88.5, 85.6), turned to 180 degrees
- moved DL14 103.4 mm to (88.6, 104.8), turned to 180 degrees
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Connections:
- U2 pad 1: ROW0_L -> (no net)
- U2 pad 10: COL3_L -> (no net)
- U2 pad 11: COL2_L -> (no net)
- U2 pad 12: VCC_L -> (no net)
- U2 pad 13: GND_L -> (no net)
- U2 pad 14: unconnected-(U2-Pad14) -> (no net)
- U2 pad 15: unconnected-(U1-Pad15) -> (no net)
- U2 pad 16: unconnected-(U1-Pad16) -> (no net)
- U2 pad 17: RESET_L -> (no net)
- U2 pad 18: GND_L -> (no net)
- U2 pad 19: BAT+_L -> (no net)
- U2 pad 2: ROW1_L -> (no net)
- U2 pad 20: GND_L -> (no net)
- U2 pad 3: ROW2_L -> (no net)
- U2 pad 4: ROW3_L -> (no net)
- U2 pad 5: COL0_L -> (no net)
- U2 pad 6: COL1_L -> (no net)
- U2 pad 7: TX_L -> (no net)
- U2 pad 8: RX_L -> (no net)
- U2 pad 9: COL4_L -> (no net)
Routing:
- net (no net): track 0.00 -> 185.8 mm, vias 0 -> 3
- net ROW0_R: track 153.3 -> 263.8 mm, vias 0 -> 10
- net ROW1_R: track 197.2 -> 297.2 mm, vias 2 -> 14
- net ROW1_L: track 247.0 -> 150.1 mm
- net ROW0_L: track 213.5 -> 130.5 mm, vias 1 -> 0
- net COL2_L: track 168.6 -> 244.4 mm, vias 2 -> 3
- net COL3_R: track 99.3 -> 161.7 mm, vias 1 -> 7
- net COL3_L: track 134.3 -> 196.3 mm, vias 1 -> 4
- net ROW3_R: track 159.6 -> 105.0 mm, vias 1 -> 4
- net COL1_R: track 143.0 -> 192.1 mm, vias 5 -> 8
- net COL2_R: track 119.6 -> 168.2 mm, vias 3 -> 7
- net COL0_R: track 187.3 -> 234.8 mm
- net COL4_R: track 81.4 -> 121.8 mm, vias 1 -> 6
- net ROW2_R: track 211.1 -> 171.0 mm, vias 2 -> 4
- net ROW3_L: track 108.8 -> 77.6 mm, vias 2 -> 0
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Other:
- board size 242.8 x 99.3 mm -> 130.4 x 102.9 mm
- board text added: "If left side solder this jumpers"
- board text added: "If right side solder this jumpers"
- board text added: "rst L"
- board text added: "rst R"
- board text removed: "pulso keyboard rev 0.2"
