File: totem swoop/totem swoop.kicad_pcb (KiCad board)
At the start: 2 copper layers, 230.9 x 97.8 mm, 141 parts, among them SW1 MX, SW17 MX, SW18 MX, SW3 SW_PUSH, U2 xiao-ble

Commit message: Add files via upload
Routing:
- net GND_R: track 159.6 -> 185.5 mm, vias 3 -> 4
- net GND_L: track 168.6 -> 176.5 mm
- net COL0_L: track 185.1 -> 192.1 mm
- net COL1_L: track 160.7 -> 165.6 mm
- net COL0_R: track 158.3 -> 160.2 mm
- net COL1_R: track 163.9 -> 164.9 mm

Commit message: Add files via upload
Parts:
- removed the BT1 at (108.8, 111.9)
- removed the BT1 at (180.8, 111.9)
- added BT1: Device_Battery_Cell, pierce:BatteryHolder_Keystone_3034_1x20mm, F.Cu at (108.9, 111.9)
- added BT1: Device_Battery_Cell, pierce:BatteryHolder_Keystone_3034_1x20mm, F.Cu at (180.9, 111.9)
- moved DL8 0.65 mm to (193.9, 77.2)
- moved DL14 0.52 mm to (212.8, 102.6)
Connections:
- SW3 pad : COL2_R -> (no net)
Routing:
- net VBAT_L: track 142.1 -> 148.0 mm, vias 2 -> 3
- net Net-(DR17-Pad2): track 35.5 -> 40.5 mm
- net GND_L: track 176.5 -> 180.5 mm, vias 2 -> 3
- net GND_R: track 185.5 -> 187.4 mm, vias 4 -> 5
- net VBAT_R: track 134.2 -> 135.7 mm, vias 3 -> 4
- net unconnected-(PSW1-Pad1): track 0.00 -> 1.50 mm
- net ROW1_L: track 111.7 -> 112.8 mm
- net ROW2_L: track 141.0 -> 141.7 mm
- net Net-(DL14-Pad2): track 15.8 -> 16.4 mm
Other:
- board text added: "Totem Swoop rev 0.1"
- board text removed: "pulso keyboard rev 0.2"

Commit message: Add files via upload
Parts:
- removed SW3 (x31): SW_PUSH, keyswitches:Kailh_socket_PG1350_reversible
Routing:
- net ROW1_R: track 156.0 -> 135.3 mm, vias 2 -> 4
- net Net-(DL18-Pad2): track 35.1 -> 23.1 mm
- net COL3_L: track 145.2 -> 133.6 mm
- net Net-(DR17-Pad2): track 40.5 -> 30.5 mm, vias 2 -> 1
- net COL4_L: track 121.5 -> 111.7 mm
- net ROW2_R: track 172.4 -> 162.8 mm
- net Net-(DR2-Pad2): track 25.1 -> 16.0 mm, vias 2 -> 1
- net Net-(DR19-Pad2): track 15.3 -> 6.75 mm, vias 2 -> 1
- net COL1_R: track 164.9 -> 158.1 mm
- net COL4_R: track 86.6 -> 79.8 mm
- net COL3_R: track 101.5 -> 94.9 mm
- net COL2_L: track 168.8 -> 162.4 mm
- net COL2_R: track 120.2 -> 113.8 mm
- net ROW1_L: track 112.8 -> 118.5 mm
- net Net-(DR15-Pad2): track 20.2 -> 14.9 mm, vias 2 -> 1
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