File: totem swoop/case/_autosave-bottom cut.kicad_pcb (KiCad board)
At the start: 2 copper layers, 114 x 97.8 mm, 13 parts

Commit message: Add files via upload
Parts:
- moved G*** 121.2 mm to (222.4, 67.6)
- moved ? 80.9 mm to (229.7, 114.0)
Changed lines of the file:
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@@
   )
   (footprint "LOGO" (layer "F.Cu")
-    (at 164.13 66.79 -90)
+    (at 229.747352 114.046487 -90)
     (attr board_only exclude_from_pos_files exclude_from_bom)
     (fp_text reference "" (at 0 0 90) (layer "Edge.Cuts")
@@
   )
   (footprint "LOGO" (layer "F.Cu")
-    (at 102.802815 87.525114)
+    (at 222.372815 67.595114)
     (attr board_only exclude_from_pos_files exclude_from_bom)
     (fp_text reference "G***" (at 0 0) (layer "F.SilkS")
